File: KiCad/A1200_IDE_LED_fix_board.kicad_pcb (KiCad board)
At the start: 2 copper layers, 45 x 15 mm, 4 parts, among them J1 Conn_02x22_Odd_Even, J2 Conn_02x22_Odd_Even, U1 74HCT2G14

Commit message: added OSHW silkscreen symbol
Parts:
- added REF**: OSHW-Symbol_6.7x6mm_SilkScreen, Symbol:OSHW-Symbol_6.7x6mm_SilkScreen, B.Cu at (129.0, 92.5)
- added REF**: OSHW-Symbol_6.7x6mm_SilkScreen, Symbol:OSHW-Symbol_6.7x6mm_SilkScreen, B.Cu at (155.0, 92.5)
